File: firmware/Atmos.kicad_sch (KiCad schematic)
At the start: 73 parts, among them J1 AS3935 breakout, J2 BME280 breakout, J3 USB_C_Receptacle_USB2.0_16P, J4 Micro_SD_Card, J5 Solar power input, J6 Conn_Coaxial, Q1 PMOS_Substrate, Q2 PMOS_Substrate, Q3 PMOS_Substrate, SW2 SW_Push, U1 ESP32-S3-WROOM-1, U10 TPS22918DBVR, U11 MAX17048G_T10, U12 CN3791, U13 SGP40-D-R4, U2 AP2112K-3.3, U3 DS3231M, U4 PMS5003, U5 LTC4412xS6, U7 RFM95W-915S2, U8 USBLC6-2SC6, U9 TPS61023DRLR

Commit message: J6: specify SMA jack (Amphenol 132134) for LoRa antenna
Parts:
- J6: value Conn_Coaxial -> Amphenol 132134
Changed lines of the file:
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@@
 			)
 		)
-		(property "Value" "Conn_Coaxial"
+		(property "Value" "Amphenol 132134"
 			(at 262.89 160.9969 0)
 			(effects
@@
 			)
 		)
-		(property "Datasheet" "~"
+		(property "Datasheet" "https://www.amphenolrf.com/132134.html"
 			(at 266.7 162.56 0)
 			(effects
@@
 			)
 		)
-		(property "Description" "coaxial connector (BNC, SMA, SMB, SMC, Cinch/RCA, LEMO, ...)"
+		(property "Description" "SMA coaxial jack, 50 ohm, vertical PCB through-hole (LoRa antenna)"
 			(at 266.7 162.56 0)
 			(effects
